File: Multi-Duino.kicad_sch (KiCad schematic)
At the start: 42 parts, among them J1 M20-9980345, J10 Micro_SD_Card_Det1, J2 M20-9980245, J8 USB_C_Receptacle_USB2.0_16P, SW1 SW_DIP_x01, U3 ATMEGA16U2-MU, U6 74LVC125, U7 DS3231MZ, U8 AT24CS32-SSHM, U9 23AA02M-ISN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

Commit message: Update Multiduino v2 design
Parts:
- removed FID1, FID2, FID3: Fiducial, Fiducial:Fiducial_1mm_Mask2mm, symbol Mechanical:Fiducial

Commit message: Update Multiduino v2 design
Parts:
- JP3, JP4, JP5: footprint (none) -> Jumper:SolderJumper-2_P1.3mm_Open_Pad1.0x1.5mm
Changed lines of the file:
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@@
 			)
 		)
-		(property "Footprint" ""
+		(property "Footprint" "Jumper:SolderJumper-2_P1.3mm_Open_Pad1.0x1.5mm"
 			(at 284.48 212.09 0)
 			(effects
@@
 			)
 		)
-		(property "Footprint" ""
+		(property "Footprint" "Jumper:SolderJumper-2_P1.3mm_Open_Pad1.0x1.5mm"
 			(at 284.48 217.17 0)
 			(effects
@@
 			)
 		)
-		(property "Footprint" ""
+		(property "Footprint" "Jumper:SolderJumper-2_P1.3mm_Open_Pad1.0x1.5mm"
 			(at 284.48 214.63 0)
 			(effects
